File: Hardware/Hardware.sch (KiCad schematic (older format))
At the start: 1 part

Commit message: Actualización Hardware
Parts:
- removed A?: Arduino_Nano_v3.x, Module:Arduino_Nano, symbol MCU_Module:Arduino_Nano_v3.x
- added C? (x2): 1uF, symbol Device:C
- added C?: 4.7uF_16V, symbol Device:CP
- added C?: 100nF, symbol Device:C
- added J?: TTL_USB, symbol Connector_Generic:Conn_01x05
- added J?: DC_DC+, symbol Connector_Generic:Conn_01x01
- added J?: DC_DC-, symbol Connector_Generic:Conn_01x01
- added J? (x2): Alarm, symbol Connector_Generic:Conn_01x02
- added J?: AudioJackPOut, symbol Connector:AudioJack3
- added J?: AudioJackF1, symbol Connector:AudioJack3
- added J?: AudioJackPIn, symbol Connector:AudioJack3
- added J?: AudioJackF2, symbol Connector:AudioJack3
- added J?: AudioJackCO2, symbol Connector:AudioJack3
- added R?: 10K, symbol Device:R
- added SW?: Button_RESET, symbol Switch:SW_Push_Dual_x2
- added U?: ATmega328P-PU, Package_DIP:DIP-28_W7.62mm, symbol MCU_Microchip_ATmega:ATmega328P-PU
- added Y?: 16MHz, symbol Device:Crystal
Connections:
- net +5V: now also C?.1, C?.1, C?.1, J?.1 (Pin_1), J?.2 (Pin_2), J?.R, J?.R, J?.R, J?.R, J?.R, R?.1, U?.7 (VCC)
- net GND: now also C?.2, C?.2, C?.2, C?.2, J?.1 (Pin_1), J?.2 (Pin_2), J?.2 (Pin_2), J?.5 (Pin_5), J?.S, J?.S, J?.S, J?.S, J?.S, SW?.2 (D), U?.22 (GND), U?.8 (GND)
- new net: U?.10 (XTAL2/PB7), Y?.2
- new net: J?.1 (Pin_1), U?.15 (PB1)
- new net: C?.1, U?.21 (AREF)
- new net: U?.9 (XTAL1/PB6), Y?.1
- new net CO2: J?.T, U?.27 (PC4)
- new net ESC: J?.1 (Pin_1), U?.17 (PB3)
- new net RESET: R?.2, SW?.1 (C), U?.1 (~RESET~/PC6)
- new net RX: J?.3 (Pin_3), U?.2 (PD0)
- new net TX: J?.4 (Pin_4), U?.3 (PD1)
- new net flow1: J?.T, U?.25 (PC2)
- new net flow2: J?.T, U?.26 (PC3)
- new net pressureIn: J?.T, U?.23 (PC0)
- new net pressureOut: J?.T, U?.24 (PC1)
- no-connect marks 3 -> 12
